File: buck_test/buck_test.kicad_pcb (KiCad board)
At the start: 4 copper layers, 42 parts, among them J1 Conn_01x02, J2 Conn_01x02, J3 Conn_01x02, J4 Conn_01x02, J5 Conn_01x02, J6 Conn_01x02, J7 Conn_01x02, J8 Conn_01x02, U1 XL1509-ADJE1, U2 TPS62160DSG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

Commit message: finished routing
Parts:
- moved J6 146.5 mm to (204.5, 33.0), turned to 180 degrees
- moved J7 137.5 mm to (199.4, 78.4)
- moved J3 129.2 mm to (170.2, 78.7)
- moved J2 116.5 mm to (175.3, 33.0), turned to 180 degrees
- moved C8 113.8 mm to (143.9, 51.8), turned to 180 degrees
- moved J8 106.6 mm to (141.0, 78.7)
- moved C11 104.8 mm to (150.5, 54.3), turned to 90 degrees
- moved C14 103.3 mm to (146.5, 52.3), turned to 180 degrees
- moved J5 90.1 mm to (146.1, 33.0), turned to 180 degrees
- moved L2 89.3 mm to (119.0, 62.0), turned to -90 degrees
- moved J1 87.8 mm to (116.8, 33.0), turned to 180 degrees
- moved R10 85.0 mm to (149.3, 51.3), turned to 90 degrees
- moved R9 80.5 mm to (149.3, 54.3), turned to 90 degrees
- moved C13 78.6 mm to (146.7, 57.3)
- moved C2 76.2 mm to (111.7, 47.2)
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Routing:
- net Net-(C3-Pad2): track 0.00 -> 18.2 mm, vias 0 -> 2
- net /5V_{Buck2}: track 0.00 -> 6.70 mm, vias 0 -> 2
- net Net-(C11-Pad2): track 0.00 -> 4.38 mm
- net Net-(C14-Pad1): track 0.00 -> 3.73 mm
- net Net-(C14-Pad2): track 0.00 -> 3.73 mm
- net GND: track 3.58 -> 4.56 mm, vias 8 -> 27
- added copper zone on F.Cu, net /5V_{Buck1}
- added copper zone on F.Cu, net /5V_{Buck2}
- added copper zone on F.Cu, net /6V5..16V
- added copper zone on F.Cu, net /6V5..40V
- added copper zone on F.Cu, net Net-(C14-Pad2)
- added copper zone on F.Cu, net Net-(D1-Pad1)
Other:
- board outline added: 124.5 x 61 mm
- board text added: "-5V"
- board text added: "5V"
- board text added: "6.5..12V"
- board text added: "6.5..16V"
- board text added: "6.5..17V"
- board text added: "6.5..40V"
- board text added: "Buck Test Board Tim Goll 02/2023"
- board text added: "GND"
- board text added: "JLCJLCJLCJLC"
- board text added: "MT2492 ----- U_{in}: 4.5(6.5)..16V U_{drop}: xxx U_{out}: 5V I_{out}: 2A f: 600kHz"
- board text added: "TPS62160DSG --------- U_{in}: 3(6.5)..17V U_{drop}: xxx U_{out}: 5V (0.6..6) I_{out}: 1A f: 2.25MHz"
- board text added: "TPS62160DSG --------- U_{in}: 3(6.5)..17V-U_{out} U_{drop}: xxx U_{out}: -5V (-0.6..-6) I_{out}: 1A f: 2.25MHz"
- board text added: "XL1509-ADJE1 --------- U_{in}: 4.5(6.5)..40V U_{drop}: 1.5V U_{out}: 5V I_{out}: 3A f: 50kHz/150kHz"
